Commit message: all the stuff from the visualizer vm

File: urdf/base.urdf.xacro (robot description, xacro)
@@ -30,5 +30,5 @@
         <!-- base_footprint is a fictitious link(frame) that is on the ground right below base_link origin,
              navigation stack depends on this frame -->
-<!--        <link name="base_footprint">
+       <link name="base_footprint">
             <inertial>
                 <mass value="0.0001" />
@@ -52,5 +52,5 @@
             <parent link="base_footprint"/>
             <child link="base_link" />
-        </joint>-->
+        </joint>
         <!-- Links and Joints (i.e., the robot) -->
         <link name="base_link">
@@ -69,9 +69,8 @@
             </visual>
             <!--Optional visualization of detailed mesh-->
-            <!--
             <visual>
                 <origin xyz="0.0 0.0 -0.049" rpy="0 0 0" />
                 <geometry>
-                    <mesh filename="package://hector_tracked_vehicles_description/meshes/jasmine_ugv/jasmine_2018_chassis_low_poly_velodyne.stl" scale="0.001 0.001 0.001"/>
+                    <!-- <mesh filename="package://hector_tracked_vehicles_description/meshes/jasmine_ugv/jasmine_2018_chassis_low_poly_velodyne.stl" scale="0.001 0.001 0.001"/> -->
                 </geometry>
                 <material name="Grey" >
@@ -79,5 +78,4 @@
                 </material>
             </visual>
-            -->
             <xacro:if value="$(arg add_default_geom)">
               <xacro:jasmine_ugv_tracks t_base_size_x="${base_size_x}"  t_base_size_y="${base_size_y}" t_base_size_z="${base_size_z}" t_flipper_offset_x="${flipper_offset_x}" t_wheel_offset_y="${wheel_offset_y}" t_wheel_radius_big="${wheel_radius_big}" t_track_width="${track_width}">

File: urdf/tankbot.urdf.xacro (robot description, xacro)
@@ -3,4 +3,9 @@
     <!-- Included URDF Files -->
     <xacro:include filename="$(find tankbot)/urdf/base.urdf.xacro" />
+    <xacro:include filename="$(find tankbot)/urdf/vision_box_common.urdf.xacro" />
+    <xacro:include filename="$(find tankbot)/urdf/vision_box_dimensions_hector1.urdf.xacro" />
     <xacro:tankbot_macro />
+    <xacro:vision_box parent="base_link" box_type="hector1">
+	     <origin xyz="-0.05 0 0.11" rpy="0 0 0"/>
+    </xacro:vision_box>
 </robot>
